File: akus_bus_V0.1/akus_bus/akus_bus.kicad_sch (KiCad schematic)
At the start: 8 parts, among them J4 12V, U1 st7735 TFT 1.8, U2 SIM800L-CORE, U3 LM7805_TO220

Commit message: Add files via upload
Parts:
- removed U1: st7735 TFT 1.8, Connector_PinSocket_2.54mm:PinSocket_1x08_P2.54mm_Vertical, symbol st7735_tft_1.8:st7735_TFT_1.8
- added F1: sigorta 2A, Fuse:Fuse_Littelfuse_395Series, symbol Device:Fuse_Small
- A1: footprint Connector_PinSocket_2.54mm:PinSocket_2x16_P2.54mm_Vertical -> DeneyapKart1A:Deneyap Kart 1A
- C2, C3: footprint Capacitor_THT:CP_Radial_Tantal_D5.0mm_P5.00mm -> Capacitor_THT:CP_Radial_D5.0mm_P2.00mm
- U2: footprint SIM800L-Core-Module-KiCad-Footprint-main:SIM800L-CORE -> Sim800l:SIM800L-CORE
Connections:
- net at J4.1 (Pin_1): now also F1.1; no longer D1.2 (A)
- new net: D1.2 (A), F1.2
