File: akus_stop_V0.1/akus_stop_V0.1.kicad_sch (KiCad schematic)
At the start: 12 parts, among them J4 Solar, J5 Li-On Şarj Devresi IN, U1 LM317_TO-220, U2 SIM800L-CORE

Commit message: c
Parts:
- C1: footprint (none) -> Capacitor_THT:CP_Radial_D4.0mm_P1.50mm
- J4: footprint (none) -> TerminalBlock:TerminalBlock_Altech_AK300-2_P5.00mm
- RV1: footprint (none) -> Potentiometer_THT:Potentiometer_ACP_CA9-H2,5_Horizontal
Changed lines of the file:
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@@
       (effects (font (size 1.27 1.27)) (justify left))
     )
-    (property "Footprint" "" (at 178.7652 58.42 0)
+    (property "Footprint" "Capacitor_THT:CP_Radial_D4.0mm_P1.50mm" (at 178.7652 58.42 0)
       (effects (font (size 1.27 1.27)) hide)
     )
@@
       (effects (font (size 1.27 1.27)))
     )
-    (property "Footprint" "" (at 196.85 58.42 0)
+    (property "Footprint" "Potentiometer_THT:Potentiometer_ACP_CA9-H2,5_Horizontal" (at 196.85 58.42 0)
       (effects (font (size 1.27 1.27)) hide)
     )
@@
       (effects (font (size 1.27 1.27)))
     )
-    (property "Footprint" "" (at 151.13 46.99 0)
-      (effects (font (size 1.27 1.27)) hide)
-    )
+    (property "Footprint" "TerminalBlock:TerminalBlock_Altech_AK300-2_P5.00mm" (at 151.13 46.99 0)
+      (effects (font (size 1.27 1.27)) hide)
+    )
